File: fonte.brd (EAGLE design)
At the start: 160 x 100 mm, 14 parts, among them T1 BC337

Commit message: Add files via upload
Parts:
- moved R2 58.9 mm to (10.2, 49.5)
- moved D5 58.4 mm to (8.89, 31.8)
- moved D2 58.3 mm to (10.2, 64.8)
- moved T1 57.1 mm to (52.1, 24.1), turned to 90 degrees
- moved R3 43.3 mm to (34.3, 12.7)
- moved JP2 40.4 mm to (52.1, 39.4), turned to 90 degrees
- moved R4 37.1 mm to (38.1, 49.5)
- moved C1 35.9 mm to (71.1, 66.0)
- moved LED1 35.6 mm to (71.1, 31.8)
- moved D1 19.4 mm to (40.6, 64.8)
- moved JP1 17.3 mm to (25.4, 91.4)
- moved R1 15.7 mm to (64.8, 49.5)
- moved D4 8.03 mm to (10.2, 78.7)
- moved D3 6.84 mm to (40.6, 78.7)
Connections:
- net N$3: now also JP2.2
- net N$4: no longer JP2.1
- net N$9: now also JP2.1; no longer JP2.2
Routing:
- net N$3: track 83.5 -> 115.7 mm
- net N$6: track 72.8 -> 43.8 mm
- net N$5: track 42.0 -> 64.2 mm
- net N$1: track 35.8 -> 53.8 mm
- net N$2: track 19.9 -> 32.2 mm
- net N$7: track 25.9 -> 19.1 mm
- net N$9: track 16.1 -> 12.7 mm
- net N$8: track 23.8 -> 20.9 mm
- net N$4: track 184.2 -> 183.0 mm

Commit message: Add files via upload
Parts:
- C1: value 330uF -> 470uF
Changed lines of the file:
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@@
 </autorouter>
 <elements>
-<element name="C1" library="rcl" library_urn="urn:adsk.eagle:library:334" package="E3,5-10" package3d_urn="urn:adsk.eagle:package:23351/1" value="330uF" x="71.12" y="66.04" smashed="yes">
+<element name="C1" library="rcl" library_urn="urn:adsk.eagle:library:334" package="E3,5-10" package3d_urn="urn:adsk.eagle:package:23351/1" value="470uF" x="71.12" y="66.04" smashed="yes">
 <attribute name="NAME" x="75.184" y="69.469" size="1.27" layer="25" ratio="10"/>
 <attribute name="POPULARITY" value="5" x="109.22" y="59.69" size="1.778" layer="27" display="off"/>
