File: fonte.sch (EAGLE design)
At the start: 14 parts, among them T1 BC337

Commit message: Add files via upload
Connections:
- net N$3: now also JP2.2
- net N$4: no longer JP2.1
- net N$9: now also JP2.1; no longer JP2.2
Changed lines of the file:
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@@
 <pinref part="D1" gate="1" pin="ANODE"/>
 <pinref part="D3" gate="1" pin="ANODE"/>
+<pinref part="JP2" gate="G$1" pin="2"/>
+<wire x1="157.48" y1="50.8" x2="198.12" y2="50.8" width="0.1524" layer="91"/>
+<wire x1="198.12" y1="50.8" x2="198.12" y2="73.66" width="0.1524" layer="91"/>
+<junction x="157.48" y="50.8"/>
 </segment>
 </net>
@@
 <junction x="137.16" y="88.9"/>
 <pinref part="T1" gate="G$1" pin="C"/>
-<pinref part="JP2" gate="G$1" pin="1"/>
-<wire x1="172.72" y1="88.9" x2="198.12" y2="88.9" width="0.1524" layer="91"/>
-<wire x1="198.12" y1="88.9" x2="198.12" y2="76.2" width="0.1524" layer="91"/>
-<junction x="172.72" y="88.9"/>
 <pinref part="D2" gate="1" pin="CATHODE"/>
 <pinref part="D4" gate="1" pin="CATHODE"/>
@@
 <segment>
 <pinref part="T1" gate="G$1" pin="E"/>
-<pinref part="JP2" gate="G$1" pin="2"/>
-<wire x1="172.72" y1="63.5" x2="198.12" y2="63.5" width="0.1524" layer="91"/>
-<wire x1="198.12" y1="63.5" x2="198.12" y2="73.66" width="0.1524" layer="91"/>
+<wire x1="172.72" y1="63.5" x2="185.42" y2="63.5" width="0.1524" layer="91"/>
+<wire x1="185.42" y1="63.5" x2="185.42" y2="76.2" width="0.1524" layer="91"/>
+<pinref part="JP2" gate="G$1" pin="1"/>
+<wire x1="185.42" y1="76.2" x2="198.12" y2="76.2" width="0.1524" layer="91"/>
 </segment>
 </net>

Commit message: Add files via upload
Parts:
- C1: value 330uF -> 470uF
Changed lines of the file:
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@@
 <part name="JP1" library="pinhead" library_urn="urn:adsk.eagle:library:325" deviceset="PINHD-1X2" device="" package3d_urn="urn:adsk.eagle:package:22435/2"/>
 <part name="JP2" library="pinhead" library_urn="urn:adsk.eagle:library:325" deviceset="PINHD-1X2" device="" package3d_urn="urn:adsk.eagle:package:22435/2"/>
-<part name="C1" library="rcl" library_urn="urn:adsk.eagle:library:334" deviceset="CPOL-EU" device="E3.5-10" package3d_urn="urn:adsk.eagle:package:23351/1" value="330uF"/>
+<part name="C1" library="rcl" library_urn="urn:adsk.eagle:library:334" deviceset="CPOL-EU" device="E3.5-10" package3d_urn="urn:adsk.eagle:package:23351/1" value="470uF"/>
 <part name="R1" library="rcl" library_urn="urn:adsk.eagle:library:334" deviceset="R-US_" device="0309/12" package3d_urn="urn:adsk.eagle:package:23571/1" value="1K"/>
 <part name="R2" library="rcl" library_urn="urn:adsk.eagle:library:334" deviceset="R-US_" device="0309/12" package3d_urn="urn:adsk.eagle:package:23571/1" value="1,8K"/>
